File: SMDModelF/SMDModelF.kicad_pcb (KiCad board)
At the start: 2 copper layers, 158.4 x 41.7 mm, 45 parts, among them J1 Model F Ribbon Cable, J2 PadsToShort, J3 EXPANSION HEADER, J4 3178 Ribbon Cable, J6 MODEL F AT LOCKLIGHTS HEADER, U1 MCP4921-E, U2 LM339A, U3 74AHC595, U4 74AHC595, U5 ProMicro, U6 LM339A

Commit message: Updated PCB file now everything points to correct 3d models.
Parts:
- J3: footprint Connector_PinHeader_2.54mm:PinHeader_2x03_P2.54mm_Vertical -> TH-XWhatsIt:PinHeader_2x03_P2.54mm_Vertical_3dhorizontal
